File: pcb-noeud/Seeeduino LoRaWan.brd (EAGLE design)
At the start: 68.6 x 53.3 mm, 111 parts, among them J4 USB / 320010000, Q1 CJ2102, Q2 CJ2101, Q3 CJ2102, Q4 CJ2101, U10 ETA6003, U3 AS179_92LF, U4 RHF76-052AM, U5 ATSAMD21G18-QFN48, U6 XC6206MR-3.3V, U7 XC6206MR-3.3V, U8 XC6206MR-3.3V, X1 32.768kHz

Commit message: Final PCB
Parts:
- removed ANT: 321050326/16cm Wire Antenna, Connector:1P-65/35MIL
- removed ANT2: U.FL, Connector-update:U-FL3P-SMD-2.6X2.6X1.0MM
- removed C10, C14: 1nF, Discrete:C0402
- removed C11, C12: 47pF, Discrete:C0402
- removed C15, C9: 1uF, Discrete:C0402
- removed C33, C34: DNP, Discrete:C0402
- removed C35, C36, C37, C38: 10uF, Discrete:C0603
- removed C39: 22uF/10v, Discrete-smallsmall:AVX-A
- removed C40: 100nF, Discrete:C0402
- removed C41: 12pF, Discrete:C0402
- removed CHG: RED, Discrete:LED-0603
- removed D5, D6: DNP, Discrete-new:SOD-923
- removed D7, D8: 1N4148WT, Discrete:SOD523
- removed DEBUG: DNP, Connector:MICRO-USB
- removed DFU: BUTTON / 311020045, Discrete-new:SW4P-SMD-4.5X3.2X2.5MM
- removed F2: DNP, Discrete-smallsmall:R0805
- removed L3: 2.2uH, Discrete:L0805
- removed LED1: DNP, Discrete:LED-0603
- removed Q4: CJ2101, Discrete:SOT323
- removed R11, R12, R15, R18, R26: 1k, Discrete:R0402
- removed R20, R22, R27, R28, R29, R44, R45, R46, R48, R50, R56: DNP, Discrete:R0402
- removed R30, R31, R47, R53: 0R, Discrete:R0402
- removed R49: 1M, Discrete:R0402
- removed R51, R52: 10k, Discrete:R0402
- removed R54, R55: 2k, Discrete:R0402
- removed R57: 1M_1%, Discrete:R0402
- removed R58: 100k_1%, Discrete:R0402
- removed T/R: YELLOW, Discrete:LED-0603
- removed U10: ETA6003, AMLib_New:QFN16G-0.5-3X3MM
- removed U3: AS179_92LF, AMLib_New:SC-70
- removed U4: RHF76-052AM, LoraWan:MODULE33P-SMD-2.0-28X23X2.9MM
- removed VBAT: DNP, Discrete:TP_4545
- added ANT1: U.FL, Connector-update:U-FL3P-SMD-2.6X2.6X1.0MM
- added ANT3: 321050326/16cm Wire Antenna, Connector:1P-65/35MIL
- added C1: 1uF, Discrete:C0603
- added C2: 4.7uF, Discrete:C0603
- added C3: 4.7F, Discrete:C0603
- added I2C2: GROVE-DIP, Connector:4P-2.0
- added R1, R2, R3, R4, R5, R6, R7: 1k, Discrete:R0603
- added SOL: 2.0 SMD JST, Connector-update:HW2-SMD-2.0-90D
- added U1: MICROCHIP_MCP73123-22SI-MFMICROCHIP_MCP73123-22SI-MF_0_0, PMIC:MICROCHIP_MCP73123-22SI-MF_0
- added U2: RF-LORA-868-SO, LoRa:XCVR_RF-LORA-868-SO
- C13, C16, C17, C18, C19, C20, C21, C22, C23, C24, C25, C26, C27, C29, C30, C31, C32: device Discrete:C0402 -> Discrete:C0603
- F1: device Discrete-smallsmall:R0805 -> Discrete-smallsmall:R0603
- R32, R33, R34, R35, R36, R37, R38, R39, R40, R41, R42, R43: device Discrete:R0402 -> Discrete:R0603
- moved BAT 18.8 mm to (58.5, 3.81), turned to 0 degrees
- moved D2 12.3 mm to (44.7, 26.9)
- moved C22 7.59 mm to (44.1, 29.6)
- moved C13 6.30 mm to (11.7, 45.7), turned to 180 degrees
- moved R34 5.16 mm to (49.4, 47.5), turned to 180 degrees
- moved C20 5.02 mm to (41.1, 48.7), turned to 0 degrees
- moved PWR 4.83 mm to (61.1, 48.3)
- moved C28 4.76 mm to (30.1, 45.5), turned to 180 degrees
- moved R41 4.49 mm to (46.9, 18.3)
- moved R36 4.32 mm to (61.1, 44.8)
- moved L 4.29 mm to (58.9, 48.3)
- moved X1 4.05 mm to (35.3, 35.9)
- moved C29 3.98 mm to (48.1, 10.8)
- moved RX 3.80 mm to (56.7, 48.3)
- moved C30 3.70 mm to (40.9, 11.0)
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Connections:
- removed net !CH_STATU: D7.-, R51.1, U10.9
- removed net DFU: C15.2, DFU.3, DFU.4, R28.2, U4.14
- removed net GNDA: C21.2, R30.2, U5.5
- removed net HF: C10.1, R15.2, U3.6
- removed net LED1: R27.1, U4.21
- removed net LED2: R26.1, U4.16
- removed net LF: C14.2, R18.2, U3.4
- removed net LORA_!RESET: D8.-, R29.1
- removed net LORA_DM: R44.2, U4.10
- removed net LORA_DP: R45.2, U4.11
- removed net LORA_SWCLK: U4.13
- removed net LORA_SWDIO: U4.12
- removed net L_RST: C15.1, D8.+, U4.27
- removed net N$21: R48.1, R53.2, U10.7
- removed net N$22: R55.2, U10.11
- removed net N$25: C34.2, D6.1, DEBUG.2, R44.1
- removed net N$26: C12.2, U3.5
- removed net N$27: C11.2, U4.32
- removed net N$28: C13.2, U4.30
- removed net N$31: R54.2, U10.12
- removed net N$33: R47.1, U10.5
- removed net N$35: R11.2, U4.4
- removed net N$36: R12.2, U4.5
- removed net N$37: CHG.-, R51.2
- removed net N$38: Q4.3, R56.1, R57.1
- removed net N$39: R20.1, U4.25
- removed net N$40: R22.1, U4.24
- removed net N$46: R26.2, T/R.-
- removed net N$48: LED1.-, R27.2
- removed net N$51: R15.1, U4.28
- removed net N$52: R18.1, U4.26
- removed net N$54: D7.+, Q4.1, R49.1, R50.1, R52.1
- removed net N$55: C11.1, U3.1
- removed net N$56: C13.1, U3.3
- removed net N$57: ANT.1, ANT2.D, C12.1
- removed net N$84: L3.1, U10.3, U10.4
- removed net PA30_SWCLK: R12.1, U5.45
- removed net PA31_SWDIO: R11.1, U5.46
- removed net U5V: C35.2, C36.2, C37.2, F1.2, F2.2, R46.1, R48.2, U10.2
- removed net VDDA: C21.1, R31.2, U5.6
- new net D0/RX_PA11_TCC0-W3: R5.1, U5.16
- new net D1/TX_PA10_TCC0-W2: R6.1, U5.15
- new net D10_SS: R4.1, U5.27
- new net D11_MOSI: R2.1, U5.25
- new net D12_MISO: R1.1, U5.28
- new net N$11: ANT1.D, ANT3.1, C13.1
- new net N$13: R2.2, U2.15
- new net N$14: R3.2, U2.13
- new net N$16: R5.2, U2.4
- new net N$17: R6.2, U2.5
- new net N$18: R7.1, U1.10
- new net N$20: U2.12
- new net N$3: C13.2, U2.1
- new net N$6: R1.2, U2.14
- net 3V3: now also BAT.+, C21.1, U5.6; no longer R31.1, R50.2
- net A4_PA05_AIN5/VBAT: no longer C41.1, R57.2, R58.1
- net A5_PB02_AIN10/!CHSTATU: no longer R52.2
- net D13_SCK: now also R3.1, U5.26
- net D32/SDA/PA22: now also I2C2.2; no longer R20.2
- net D33/SCL/PA23: now also I2C2.1; no longer R22.2
- net D8_DGI_GPIO2/LORA_!RST: no longer R29.2
- net D9_DGI_GPIO3/LORA_DFU: no longer R28.1
- net GND: now also ANT1.GND1, ANT1.GND2, C1.2, C2.1, C21.2, C3.2, I2C2.4, R7.2, SOL.-, SOL.3, SOL.4, U1.11, U1.8, U1.9, U2.2, U5.5; no longer ANT2.GND1, ANT2.GND2, C10.2, C14.1, C33.1, C34.1, C35.1, C36.1, C37.1, C38.1, C39.-, C40.1, C41.2, C9.2, D5.2, D6.2, DEBUG.5, DEBUG.S1, DEBUG.S2, DEBUG.S3, DEBUG.S4, DEBUG.S5, DEBUG.S6, DFU.1, DFU.2, R30.1, R47.2, R53.1, R54.1, R55.1, R58.2, U10.10, U10.13, U10.6, U10.8, U10.PAD, U3.2, U4.2, U4.29, U4.31, U4.33
- net GROVE_3V3: now also I2C2.3
- net LIPO_BAT: now also C2.2, U1.3, U1.4; no longer BAT.+, C40.2, Q4.2, R56.2, U10.14, U10.16, VBAT.T
- net LORA_3V3: no longer C9.1, LED1.+, T/R.+, U4.1
- net N$15: now also R4.2, U2.16; no longer DEBUG.1, F2.1
- net N$9: now also C1.1, U2.3; no longer C33.2, D5.1, DEBUG.3, R45.1
- net VIN: now also C3.1, F1.2, SOL.+, U1.1, U1.2; no longer C38.2, C39.+, CHG.+, L3.2, R46.2, R49.2, U10.1, U10.15
Routing:
- net L_RST: track 72.0 -> 0.00 mm, vias 4 -> 0
- net A4_PA05_AIN5/VBAT: track 69.4 -> 0.00 mm, vias 4 -> 0
- net D8_DGI_GPIO2/LORA_!RST: track 50.0 -> 0.00 mm, vias 4 -> 0
- net D1/TX_PA10_TCC0-W2: track 0.00 -> 47.6 mm, vias 0 -> 4
- net D0/RX_PA11_TCC0-W3: track 0.00 -> 46.9 mm, vias 0 -> 4
- net DFU: track 46.7 -> 0.00 mm, vias 4 -> 0
- net 3V3: track 90.2 -> 135.5 mm, vias 12 -> 14
- net D10_SS: track 0.00 -> 40.5 mm, vias 0 -> 4
- net PA31_SWDIO: track 38.2 -> 0.00 mm, vias 3 -> 0
- net U5V: track 37.7 -> 0.00 mm, vias 4 -> 0
- net D13_SCK: track 1.48 -> 38.5 mm, vias 0 -> 3
- net LORA_3V3: track 45.3 -> 8.39 mm, vias 2 -> 0
- net LORA_DM: track 36.7 -> 0.00 mm, vias 2 -> 0
- net LORA_DP: track 36.5 -> 0.00 mm, vias 2 -> 0
- net D11_MOSI: track 0.00 -> 35.9 mm, vias 0 -> 2
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- removed copper zone on layer 16, net N$84
- removed copper zone on layer 16, net VIN
Other:
- board text removed: "CHG"
- board text removed: "D10"
- board text removed: "DFU"
- board text removed: "R"
- board text removed: "S"

Commit message: Added gateway files
Parts:
- C3: value 4.7F -> 4.7uF
Connections:
- removed net N$9: C1.1, U2.3
- net LORA_3V3: now also C1.1, U2.3
Routing:
- net LORA_3V3: track 8.39 -> 42.0 mm, vias 0 -> 4
- net N$9: track 3.37 -> 0.00 mm
Changed lines of the file:
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@@
 <?xml version="1.0" encoding="utf-8"?>
 <!DOCTYPE eagle SYSTEM "eagle.dtd">
-<eagle version="9.3.1">
+<eagle version="9.3.2">
 <drawing>
 <settings>
@@
 </layers>
 <board>
+<fusionsync huburn="a.cGVyc29uYWw6dWUyOWE3NWEy" projecturn="a.cGVyc29uYWw6dWUyOWE3NWEyIzIwMTUwNjI1MTQwMTg0MzE" f3durn="urn:adsk.wipprod:dm.lineage:mxmJGioOTrCV8BumaUHFwg" pcbguid="cdbe6112-0e97-4e38-80e3-706cc3e83e13" lastpulledtime="" lastsyncedchangeguid="883bd00f-16fe-26c9-6d9b-bcba92bcc3f5"/>
 <plain>
 <wire x1="68.58" y1="52.07" x2="67.31" y2="53.34" width="0.0254" layer="20" curve="90"/>
@@
 </element>
 <element name="ANT3" library="Connector" package="1P-65/35MIL" value="321050326/16cm Wire Antenna" x="3.556" y="42.418" smashed="yes">
-<attribute name="NAME" x="5.207" y="41.148" size="0.8128" layer="25"/>
+<attribute name="NAME" x="4.445" y="40.894" size="0.8128" layer="25"/>
 </element>
 <element name="R1" library="Discrete" package="R0603" value="1k" x="21.12433125" y="43.053" smashed="yes" rot="MR270">
@@
 <attribute name="VALUE" x="61.087" y="15.0495" size="0.381" layer="28" ratio="12" rot="MR0"/>
 </element>
-<element name="C3" library="Discrete" package="C0603" value="4.7F" x="59.817" y="18.034" smashed="yes" rot="MR180">
+<element name="C3" library="Discrete" package="C0603" value="4.7uF" x="59.817" y="18.034" smashed="yes" rot="MR180">
 <attribute name="NAME" x="58.42" y="17.272" size="0.889" layer="26" ratio="11" rot="MR180"/>
 <attribute name="NAME" x="58.547" y="18.288" size="0.635" layer="34" ratio="10" rot="MR180"/>
@@
 <wire x1="37.6335" y1="46.46" x2="36.449" y2="46.46" width="0.1524" layer="16"/>
 <wire x1="35.262" y1="45.273" x2="31.1175" y2="45.273" width="0.1524" layer="16"/>
+<contactref element="U2" pad="3"/>
+<contactref element="C1" pad="1"/>
+<wire x1="30.734" y1="33.147" x2="30.653" y2="33.228" width="0.1524" layer="16"/>
+<wire x1="30.653" y1="33.228" x2="27.394" y2="33.228" width="0.1524" layer="16"/>
 <wire x1="31.1175" y1="45.273" x2="30.861" y2="45.5295" width="0.1524" layer="16"/>
+<wire x1="30.861" y1="45.5295" x2="31.496" y2="46.1645" width="0.1524" layer="16"/>
+<wire x1="31.496" y1="46.1645" x2="31.496" y2="46.482" width="0.1524" layer="16"/>
+<via x="31.496" y="46.482" extent="1-16" drill="0.2032" diameter="0.2032"/>
+<wire x1="31.496" y1="46.482" x2="27.559" y2="46.482" width="0.1524" layer="1"/>
+<wire x1="27.559" y1="46.482" x2="26.0604" y2="44.9834" width="0.1524" layer="1"/>
+<wire x1="25.9936625" y1="44.9834" x2="25.7556" y2="44.7453375" width="0.1524" layer="1"/>
+<wire x1="25.7556" y1="44.7453375" x2="25.7556" y2="44.704" width="0.1524" layer="1"/>
+<wire x1="26.0604" y1="44.9834" x2="25.9936625" y2="44.9834" width="0.1524" layer="1"/>
+<wire x1="19.558" y1="44.704" x2="18.796" y2="43.942" width="0.1524" layer="1"/>
+<via x="18.796" y="43.942" extent="1-16" drill="0.2032" diameter="0.2032"/>
+<wire x1="18.796" y1="43.942" x2="18.796" y2="40.132" width="0.1524" layer="16"/>
+<via x="18.796" y="40.132" extent="1-16" drill="0.2032" diameter="0.2032"/>
+<wire x1="18.796" y1="40.132" x2="24.13" y2="34.798" width="0.1524" layer="1"/>
+<via x="24.13" y="34.798" extent="1-16" drill="0.2032" diameter="0.2032"/>
+<wire x1="24.13" y1="34.798" x2="25.7" y2="33.228" width="0.1524" layer="16"/>
+<wire x1="25.7" y1="33.228" x2="27.394" y2="33.228" width="0.1524" layer="16"/>
+<wire x1="25.7556" y1="44.704" x2="19.558" y2="44.704" width="0.1524" layer="1"/>
 </signal>
 <signal name="VIN">
@@
 <wire x1="50.264" y1="43.66" x2="49.297" y2="43.66" width="0.1524" layer="16"/>
 </signal>
-<signal name="N$9">
-<contactref element="U2" pad="3"/>
-<contactref element="C1" pad="1"/>
-<wire x1="30.734" y1="33.147" x2="30.653" y2="33.228" width="0.1524" layer="16"/>
-<wire x1="30.653" y1="33.228" x2="27.394" y2="33.228" width="0.1524" layer="16"/>
-</signal>
 <signal name="N$11">
 <contactref element="ANT1" pad="D"/>
@@
 </board>
 </drawing>
+<compatibility>
+<note version="8.3" severity="warning">
+Since Version 8.3, EAGLE supports Fusion synchronisation.
+This feature will not be available in this version and saving
+the document will break the link to the Fusion PCB feature.
+</note>
+</compatibility>
 </eagle>
