File: pcb-noeud/Seeeduino LoRaWan.sch (EAGLE design)
At the start: 111 parts, among them J4 USB / 320010000, Q1 CJ2102, Q2 CJ2101, Q3 CJ2102, Q4 CJ2101, U10 ETA6003, U3 AS179_92LF, U4 RHF76-052AM, U5 ATSAMD21G18-QFN48, U6 XC6206MR-3.3V, U7 XC6206MR-3.3V, U8 XC6206MR-3.3V, X1 32.768kHz

Commit message: Final PCB
Parts:
- removed ANT: 321050326/16cm Wire Antenna, Connector:HEADER-1P-35
- removed ANT2: U.FL, Connector-update:ANTENNA-U-FL
- removed C10, C14: 1nF, Discrete:C-0402
- removed C11, C12: 47pF, Discrete:C-0402
- removed C15, C9: 1uF, Discrete:C-0402
- removed C33, C34: DNP, Discrete:C-0402
- removed C35, C36, C37, C38: 10uF, Discrete:C-0603
- removed C39: 22uF/10v, Discrete-smallsmall:CAP-AVX-A
- removed C40: 100nF, Discrete:C-0402
- removed C41: 12pF, Discrete:C-0402
- removed CHG: RED, Discrete:LED'0603'
- removed D5, D6: DNP, Discrete-new:D-ESD-2P'DF2S6.8FS'
- removed D7, D8: 1N4148WT, Discrete:D'0603'
- removed DEBUG: DNP, Connector:USB-MINIUSB-5P-MICRO
- removed DFU: BUTTON / 311020045, Discrete-new:BUTTON-4P-4.5X3.2
- removed F2: DNP, Discrete-smallsmall:R-0805
- removed L3: 2.2uH, Discrete:L'0805'
- removed LED1: DNP, Discrete:LED'0603'
- removed Q4: CJ2101, Discrete:MOSFET-P-SOT323
- removed R11, R12, R15, R18, R26: 1k, Discrete:R-0402
- removed R20, R22, R27, R28, R29, R44, R45, R46, R48, R50, R56: DNP, Discrete:R-0402
- removed R30, R31, R47, R53: 0R, Discrete:R-0402
- removed R49: 1M, Discrete:R-0402
- removed R51, R52: 10k, Discrete:R-0402
- removed R54, R55: 2k, Discrete:R-0402
- removed R57: 1M_1%, Discrete:R-0402
- removed R58: 100k_1%, Discrete:R-0402
- removed T/R: YELLOW, Discrete:LED'0603'
- removed U10: ETA6003, AMLib_New:PMIC-ETA6003
- removed U3: AS179_92LF, AMLib_New:PE4259
- removed U4: RHF76-052AM, LoraWan:MODULE-LORAWAN-RHF76-052
- removed VBAT: DNP, Discrete:PAD-TEST-POINT'4545'
- added ANT1: U.FL, Connector-update:ANTENNA-U-FL
- added ANT3: 321050326/16cm Wire Antenna, Connector:HEADER-1P-35
- added C1: 1uF, Discrete:C-0603
- added C2: 4.7uF, Discrete:C-0603
- added C3: 4.7F, Discrete:C-0603
- added I2C2: GROVE-DIP, Connector:TWIG-4P-2.0-2.0
- added R1, R2, R3, R4, R5, R6, R7: 1k, Discrete:R-0603
- added SOL: 2.0 SMD JST, Connector-update:JST-2P-SMD'2.0'
- added U1: MICROCHIP_MCP73123-22SI-MFMICROCHIP_MCP73123-22SI-MF_0_0, PMIC:MICROCHIP_MCP73123-22SI-MFMICROCHIP_MCP73123-22SI-MF_0_0
- added U2: RF-LORA-868-SO, LoRa:RF-LORA-868-SO
- C13, C16, C17, C18, C19, C20, C21, C22, C23, C24, C25, C26, C27, C29, C30, C31, C32: device Discrete:C-0402 -> Discrete:C-0603
- F1: device Discrete-smallsmall:R-0805 -> Discrete-smallsmall:R-0603
- R32, R33, R34, R35, R36, R37, R38, R39, R40, R41, R42, R43: device Discrete:R-0402 -> Discrete:R-0603
Connections:
- removed net !CH_STATU: D7.-, R51.1, U10.STAT
- removed net DFU: C15.2, DFU.B0, DFU.B1, R28.2, U4.PA15
- removed net GNDA: C21.2, R30.2, U5.GNDANA
- removed net HF: C10.1, R15.2, U3.!CTRL!/VDD
- removed net LED1: R27.1, U4.PB5
- removed net LED2: R26.1, U4.PB4
- removed net LF: C14.2, R18.2, U3.CTRL
- removed net LORA_!RESET: D8.-, R29.1
- removed net LORA_DM: R44.2, U4.USART_CTS
- removed net LORA_DP: R45.2, U4.USART_RTS
- removed net LORA_SWCLK: U4.SWCLK
- removed net LORA_SWDIO: U4.SWDIO
- removed net L_RST: C15.1, D8.+, U4.NRST
- removed net N$21: R48.1, R53.2, U10.NTC
- removed net N$22: R55.2, U10.ISET1
- removed net N$25: C34.2, D6.2, DEBUG.DM, R44.1
- removed net N$26: C12.2, U3.RFC
- removed net N$27: C11.2, U4.RFIO_LF
- removed net N$28: C13.2, U4.RFIO_HF
- removed net N$31: R54.2, U10.ISET2
- removed net N$33: R47.1, U10.PGND
- removed net N$35: R11.2, U4.PA9
- removed net N$36: R12.2, U4.PA10
- removed net N$37: CHG.-, R51.2
- removed net N$38: Q4.D, R56.1, R57.1
- removed net N$39: R20.1, U4.SDA
- removed net N$40: R22.1, U4.SCL
- removed net N$46: R26.2, T/R.-
- removed net N$48: LED1.-, R27.2
- removed net N$51: R15.1, U4.PA0
- removed net N$52: R18.1, U4.PC13
- removed net N$54: D7.+, Q4.G, R49.1, R50.1, R52.1
- removed net N$55: C11.1, U3.RF1
- removed net N$56: C13.1, U3.RF2
- removed net N$57: ANT.1, ANT2.D, C12.1
- removed net N$84: L3.1, U10.SW, U10.SW@1
- removed net PA30_SWCLK: R12.1, U5.PA30/EIC/SCOM1PAD2/TC1
- removed net PA31_SWDIO: R11.1, U5.PA31/EIC/SCOM1PAD3/TC1
- removed net U5V: C35.2, C36.2, C37.2, F1.2, F2.2, R46.1, R48.2, U10.IN
- removed net VDDA: C21.1, R31.2, U5.VDDANA
- new net D0/RX_PA11_TCC0-W3: R5.1, U5.PA11/EIC/AIN19/SCOM2PAD3+/TC1
- new net D1/TX_PA10_TCC0-W2: R6.1, U5.PA10/EIC/AIN18/SCOM2PAD2+/TC1
- new net D10_SS: R4.1, U5.PA18/EIC/SCOM1PAD2+/TC3
- new net D11_MOSI: R2.1, U5.PA16/I2C/EIC/SCOM1PAD0+/TC2
- new net D12_MISO: R1.1, U5.PA19/EIC/SCOM1PAD3+/TC3
- new net N$11: ANT1.D, ANT3.1, C13.1
- new net N$13: R2.2, U2.SDI
- new net N$14: R3.2, U2.SCLK
- new net N$16: R5.2, U2.RX_SWITCH
- new net N$17: R6.2, U2.TX_SWITCH
- new net N$18: R7.1, U1.PROG
- new net N$20: U2.RESET
- new net N$3: C13.2, U2.ANT
- new net N$6: R1.2, U2.SDO
- net 3V3: now also BAT.1, C21.1, U5.VDDANA; no longer R31.1, R50.2
- net A4_PA05_AIN5/VBAT: no longer C41.1, R57.2, R58.1
- net A5_PB02_AIN10/!CHSTATU: no longer R52.2
- net D13_SCK: now also R3.1, U5.PA17/I2C/EIC/SCOM1PAD1+/TC2
- net D32/SDA/PA22: now also I2C2.2; no longer R20.2
- net D33/SCL/PA23: now also I2C2.1; no longer R22.2
- net D8_DGI_GPIO2/LORA_!RST: no longer R29.2
- net D9_DGI_GPIO3/LORA_DFU: no longer R28.1
- net GND: now also ANT1.GND1, ANT1.GND2, C1.2, C2.1, C21.2, C3.2, I2C2.4, R7.2, SOL.2, SOL.3, SOL.4, U1.1_VSS, U1.2_VSS, U1.VSS_PAD, U2.GND, U5.GNDANA; no longer ANT2.GND1, ANT2.GND2, C10.2, C14.1, C33.1, C34.1, C35.1, C36.1, C37.1, C38.1, C39.-, C40.1, C41.2, C9.2, D5.1, D6.1, DEBUG.GND@1, DEBUG.GND@2, DEBUG.GND@3, DEBUG.GND@4, DEBUG.GND@5, DFU.A0, DFU.A1, R30.1, R47.2, R53.1, R54.1, R55.1, R58.2, U10.ENB, U10.GND, U10.GND@1, U10.PAD, U10.USB_DET, U3.GND, U4.GND, U4.GND@1, U4.GND@2, U4.GND@3
- net GROVE_3V3: now also I2C2.3
- net LIPO_BAT: now also C2.2, U1.1_VBAT, U1.2_VBAT; no longer BAT.1, C40.2, Q4.S, R56.2, U10.BATT, U10.BATT@1, VBAT.T
- net LORA_3V3: no longer C9.1, LED1.+, T/R.+, U4.VCC
- net N$15: now also R4.2, U2.!SEL; no longer DEBUG.VCC, F2.1
- net N$9: now also C1.1, U2.VCC; no longer C33.2, D5.2, DEBUG.DP, R45.1
- net VIN: now also C3.1, F1.2, SOL.1, U1.1_VDD, U1.2_VDD; no longer C38.2, C39.+, CHG.+, L3.2, R46.2, R49.2, U10.SYS, U10.SYS@1
Other:
- note added: "Custom battery management"
- note removed: "Firmware upgrade"
- note removed: "close to pin10"
- note removed: "close to pin2"
- note removed: "if no battery, led flash. if charging, led on. if charge ok, led off."
- moved on the sheet: C13

Commit message: Added gateway files
Parts:
- C3: value 4.7F -> 4.7uF
Connections:
- removed net N$9: C1.1, U2.VCC
- net LORA_3V3: now also C1.1, U2.VCC
Changed lines of the file:
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@@
 <?xml version="1.0" encoding="utf-8"?>
 <!DOCTYPE eagle SYSTEM "eagle.dtd">
-<eagle version="9.3.1">
+<eagle version="9.3.2">
 <drawing>
 <settings>
@@
 <part name="GND19" library="Power or GND " deviceset="GND_POWER" device=""/>
 <part name="GND20" library="Power or GND " deviceset="GND_POWER" device=""/>
-<part name="C3" library="Discrete" deviceset="C*" device="-0603" value="4.7F"/>
+<part name="C3" library="Discrete" deviceset="C*" device="-0603" value="4.7uF"/>
 <part name="GND12" library="Power or GND " deviceset="GND_POWER" device=""/>
 </parts>
@@
 </segment>
 <segment>
-<label x="353.06" y="297.18" size="0.889" layer="95" ratio="12" rot="MR180" xref="yes"/>
+<pinref part="U2" gate="G$1" pin="VCC"/>
+<wire x1="342.9" y1="297.18" x2="347.98" y2="297.18" width="0.1524" layer="91"/>
+<pinref part="C1" gate="C" pin="1"/>
+<wire x1="347.98" y1="297.18" x2="347.98" y2="299.72" width="0.1524" layer="91"/>
+<wire x1="347.98" y1="297.18" x2="353.06" y2="297.18" width="0.1524" layer="91"/>
+<junction x="347.98" y="297.18"/>
+<label x="353.06" y="297.18" size="0.889" layer="95" xref="yes"/>
 </segment>
 </net>
@@
 </segment>
 </net>
-<net name="N$9" class="0">
-<segment>
-<pinref part="U2" gate="G$1" pin="VCC"/>
-<wire x1="342.9" y1="297.18" x2="347.98" y2="297.18" width="0.1524" layer="91"/>
-<pinref part="C1" gate="C" pin="1"/>
-<wire x1="347.98" y1="297.18" x2="347.98" y2="299.72" width="0.1524" layer="91"/>
-<junction x="347.98" y="297.18"/>
-<wire x1="353.06" y1="297.18" x2="347.98" y2="297.18" width="0.1524" layer="91"/>
-</segment>
-</net>
